File: hw/WifiRelay.sch (KiCad schematic (older format))
At the start: 35 parts, among them J1 CONN_01X02, J2 CONN_01X06, J3 CONN_01X02, J4 CONN_01X02, J5 TEST_1P, J6 TEST_1P, K1 Songle-SRD-05VDC-SL-C, K2 Songle-SRD-05VDC-SL-C, Q1 MMSS8050-H, Q2 MMSS8050-H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

Commit message: Remapped symbols into V5 libraries
Parts:
- C1, C2: symbol CP -> device:CP
- C3, C4: symbol C -> device:C
- D1, D2: symbol 1N4148 -> WifiRelay:1N4148
- J1, J3, J4: symbol CONN_01X02 -> conn:CONN_01X02
- J2: symbol CONN_01X06 -> conn:CONN_01X06
- J5, J6: symbol TEST_1P -> conn:TEST_1P
- JP1: symbol Jumper_Dual -> WifiRelay:Jumper_Dual
- K1, K2: symbol Songle-SRD-05VDC-SL-C -> WifiRelay:Songle-SRD-05VDC-SL-C
- Q1, Q2: symbol MMSS8050-H -> transistors:MMSS8050-H
- R1, R10, R11, R12, R2, R3, R4, R5, R6, R7, R8, R9: symbol R -> device:R
- SW1, SW2: symbol SW_Push -> switches:SW_Push
- U1: symbol IRM-02-5 -> WifiRelay:IRM-02-5
- U2: symbol LM1117-3.3 -> regul:LM1117-3.3
- U3: symbol ESP-07v2 -> ESP8266:ESP-07v2
- U4: symbol PC827 -> opto:PC827
