File: hw/WifiRelay.kicad_pcb (KiCad board)
At the start: 2 copper layers, 94 x 54 mm, 35 parts, among them J1 CONN_01X02, J2 CONN_01X06, J3 CONN_01X02, J4 CONN_01X02, J5 TEST_1P, J6 TEST_1P, K1 Songle-SRD-05VDC-SL-C, K2 Songle-SRD-05VDC-SL-C, Q1 MMSS8050-H, Q2 MMSS8050-H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

Commit message: Added 3D shapes for 2 pin terminal blocks J1, J3 and J4
Parts:
- J1, J4: footprint TerminalBlock_Phoenix:TerminalBlock_Phoenix_MKDS-1,5-2_1x02_P5.00mm_Horizontal -> Connectors_Terminal_Blocks:TerminalBlock_Pheonix_MKDS1.5-2pol
Connections:
- J1 pad 1: Net-(J1-Pad1) -> (no net)
- J1 pad 2: Net-(J1-Pad2) -> (no net)
- J4 pad 1: Net-(J4-Pad1) -> (no net)
- J4 pad 2: Net-(J4-Pad2) -> (no net)

Commit message: Added 3D symbol for ESP-07. Corrected connections to J1 and J4 (broken in previous revision)
Parts:
- J1, J4: footprint Connectors_Terminal_Blocks:TerminalBlock_Pheonix_MKDS1.5-2pol -> TerminalBlock_Phoenix:TerminalBlock_Phoenix_MKDS-1,5-2_1x02_P5.00mm_Horizontal
Connections:
- J1 pad 1: (no net) -> Net-(J1-Pad1)
- J1 pad 2: (no net) -> Net-(J1-Pad2)
- J4 pad 1: (no net) -> Net-(J4-Pad1)
- J4 pad 2: (no net) -> Net-(J4-Pad2)
